File: CTS-SAT-2-Magnetometer-Module/CTS-SAT-2-Magnetometer-Module.kicad_pcb (KiCad board)
At the start: 2 copper layers, 24 x 35.5 mm, 32 parts, among them J1 PicoBlade, J2 SWD, U1 MMC5983MA, U2 LIS2MDL, U3 STM32F072C8Tx, U4 MIC5365-3.3YD5

Commit message: Re-routed
Parts:
- removed 10k1, 10k2, 3K3: R, Resistor_SMD:R_0603_1608Metric_Pad0.98x0.95mm_HandSolder
- removed D1: LED, LED_SMD:LED_0603_1608Metric_Pad1.05x0.95mm_HandSolder
- added C7: 100nF, Capacitor_SMD:C_0603_1608Metric_Pad1.08x0.95mm_HandSolder, F.Cu at (203.5, 89.4)
- added D3: LED, LED_SMD:LED_0603_1608Metric_Pad1.05x0.95mm_HandSolder, F.Cu at (188.5, 90.1)
- added D4: LED, LED_SMD:LED_0603_1608Metric_Pad1.05x0.95mm_HandSolder, F.Cu at (188.0, 102.0)
- added J3: SWD, Connector_PinHeader_2.54mm:PinHeader_1x05_P2.54mm_Vertical, F.Cu at (207.6, 104.5)
- added R7: 3K3, Resistor_SMD:R_0603_1608Metric_Pad0.98x0.95mm_HandSolder, F.Cu at (188.0, 98.1)
- added SW1: SW_Push, Button_Switch_SMD:SW_SPST_EVQP0, F.Cu at (198.0, 86.5)
- C10: renamed from 100nF3; value C -> 100nF3
- C11: renamed from 100nF4; value C -> 100nF4
- C12: renamed from 100nF5; value C -> 100nF5
- C13: renamed from 1uF1; value C -> 1uF1
- C14: renamed from 10uF1; value C -> 10uF1
- C8: renamed from 100nF1; value C -> 100nF1
- C9: renamed from 100nF2; value C -> 100nF2
- R1: value 3K3 -> 0
- R3: value 4k7 -> 10k
- R4: value 4k7 -> 3K3
- moved R3 22.5 mm to (192.5, 88.0), turned to -90 degrees
- moved G*** 18.7 mm to (171.5, 81.5)
- moved R4 17.6 mm to (188.5, 94.2), turned to 90 degrees
- moved J2 15.1 mm to (213.3, 97.8), turned to 0 degrees
- moved C8 8.24 mm to (205.5, 99.5), turned to 90 degrees
- moved R1 5.53 mm to (195.4, 111.6)
- moved D4 4.12 mm to (186.0, 107.9)
- moved U1 4.12 mm to (189.0, 108.0)
- moved C14 3.86 mm to (188.4, 111.2)
- moved C11 3.64 mm to (190.0, 102.0), turned to 90 degrees
- moved C13 3.50 mm to (187.5, 105.0), turned to 180 degrees
- moved C4 3.24 mm to (196.9, 115.6), turned to -90 degrees
- moved C1 2.02 mm to (191.9, 116.4)
- moved C3 1.85 mm to (192.1, 113.9)
- moved U2 1.85 mm to (194.4, 114.1)
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Connections:
- C1 pad 2: +3.3V -> +3V0
- C10 pad 2: +3.3V -> +3V0
- C11 pad 2: +3.3V -> +3V0
- C12 pad 1: +3.3V -> +3V0
- C13 pad 1: +3.3V -> +3V0
- C2 pad 1: +3.3V -> +3V0
- C4 pad 1: +3.3V -> +3V0
- C6 pad 1: +3.3V -> +3V0
- C8 pad 2: +3.3V -> +3V0
- C9 pad 2: +3.3V -> +3V0
- J2 pad 2: VCC -> Vdd
- J2 pad 3: RESET -> NRST
- R1 pad 1: +3.3V -> +3V0
- R1 pad 2: Net-(D1-A) -> Net-(U2-~{CS})
- R2 pad 1: +3.3V -> +3V0
- R3 pad 1: +3.3V -> +3V0
- R3 pad 2: SDA -> NRST
- R4 pad 1: +3.3V -> Net-(U3-PB0)
- R4 pad 2: SCL -> Net-(D3-A)
- R5 pad 1: +3.3V -> +3V0
- R6 pad 1: +3.3V -> +3V0
- U1 pad 13: +3.3V -> +3V0
- U1 pad 15: unconnected-(U1-INT-Pad15) -> INT
- U1 pad 2: +3.3V -> +3V0
- U1 pad 4: +3.3V -> +3V0
- U2 pad 10: +3.3V -> +3V0
- U2 pad 3: +3.3V -> Net-(U2-~{CS})
- U2 pad 7: unconnected-(U2-DRDY-Pad7) -> DRDY
- U2 pad 9: +3.3V -> +3V0
- U3 pad 1: +3.3V -> +3V0
- U3 pad 18: unconnected-(U3-PB0-Pad18) -> Net-(U3-PB0)
- U3 pad 19: unconnected-(U3-PB1-Pad19) -> Net-(U3-PB1)
- U3 pad 20: unconnected-(U3-PB2-Pad20) -> INT
- U3 pad 21: unconnected-(U3-PB10-Pad21) -> DRDY
- U3 pad 23: unconnected-(U3-VSS-Pad23) -> GND
- U3 pad 24: +3.3V -> +3V0
- U3 pad 34: unconnected-(U3-PA13-Pad34) -> SWDIO
- U3 pad 35: unconnected-(U3-VSS-Pad23)_2 -> GND
- U3 pad 36: +3.3V -> +3V0
- U3 pad 37: unconnected-(U3-PA14-Pad37) -> SWDCLK
- U3 pad 47: unconnected-(U3-VSS-Pad23)_1 -> GND
- U3 pad 48: +3.3V -> +3V0
- U3 pad 7: RESET -> NRST
- U3 pad 8: unconnected-(U3-VSSA-Pad8) -> GND
- U3 pad 9: +3.3V -> +3V0
- U4 pad 5: +3.3V -> +3V0
Routing:
- net +3.3V: track 30.5 -> 0.00 mm
- net GND: track 43.7 -> 19.0 mm, vias 15 -> 4
- net +3V0: track 0.00 -> 18.5 mm
- net SCL: track 24.0 -> 14.5 mm, vias 1 -> 0
- net SDA: track 20.5 -> 11.4 mm
- net RESET: track 5.64 -> 0.00 mm
- net SWDIO: track 0.00 -> 5.04 mm
- net Net-(D1-A): track 2.05 -> 0.00 mm
- net Net-(U2-~{CS}): track 0.00 -> 1.88 mm
- net Net-(D4-A): track 1.75 -> 0.00 mm
- removed copper zone on F.Cu, net +3.3V
- removed copper zone on B.Cu, net GND
Other:
- board outline removed
- board text removed: "Magnetometer Dev Board"
- board text removed: "Marian Abebe"
- board text removed: "Rev2.0"

Commit message: Applied Changes following Review 2
Parts:
- removed the D4 at (186.0, 107.9)
- moved J2 13.6 mm to (205.0, 108.6), turned to 180 degrees
- moved SW1 10.9 mm to (207.4, 92.0)
- moved R3 7.36 mm to (199.6, 90.0), turned to 180 degrees
- moved C7 7.00 mm to (196.5, 89.5), turned to 90 degrees
- moved C8 5.85 mm to (200.0, 101.5), turned to 180 degrees
- moved J3 4.32 mm to (209.0, 108.6), turned to 180 degrees
- moved C3 2.90 mm to (191.5, 111.0), turned to 90 degrees
- moved C9 2.06 mm to (193.0, 89.0), turned to -90 degrees
- moved D3 2.03 mm to (190.0, 91.5), turned to 180 degrees
- moved U1 1.84 mm to (188.0, 109.5)
- moved R5 1.80 mm to (195.5, 103.0), turned to 180 degrees
- moved C13 1.61 mm to (187.1, 106.5)
- moved C14 1.58 mm to (187.5, 112.5)
- moved J1 1.55 mm to (200.0, 107.4)
- moved D4 1.51 mm to (186.5, 101.9)
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Routing:
- net GND: track 19.0 -> 73.5 mm, vias 4 -> 14
- net NRST: track 0.00 -> 54.5 mm, vias 0 -> 2
- net +3V0: track 18.5 -> 57.1 mm, vias 0 -> 5
- net Vdd: track 8.21 -> 31.0 mm
- net DRDY: track 0.00 -> 20.2 mm, vias 0 -> 2
- net SWDCLK: track 0.00 -> 10.4 mm
- net SCL: track 14.5 -> 24.8 mm, vias 0 -> 2
- net SWDIO: track 5.04 -> 14.3 mm
- net SDA: track 11.4 -> 17.6 mm
- net INT: track 0.00 -> 4.21 mm, vias 0 -> 2
- net Net-(U3-PB0): track 0.00 -> 3.32 mm
- net Net-(U3-PB1): track 0.00 -> 2.87 mm
- net Net-(D4-A): track 0.00 -> 2.62 mm
- net Net-(D3-A): track 0.00 -> 2.01 mm
- net Net-(U2-C1): track 1.85 -> 2.42 mm
- added copper zone on F.Cu, net +3V0
- added copper zone on B.Cu, net GND
Other:
- board outline added: 31.5 x 37.5 mm

Commit message: First pcb multi layers
Parts:
- removed G***: LOGO, LOGO
- removed J3: SWD, Connector_PinHeader_2.54mm:PinHeader_1x05_P2.54mm_Vertical
- removed U4: MIC5365-3.3YD5, Package_TO_SOT_SMD:SOT-23-5
- added U5: MIC5365-3.0YC5, Package_TO_SOT_SMD:SOT-353_SC-70-5, F.Cu at (115.3, 152.2)
- J1: value PicoBlade -> Conn_01x04_Pin
- moved SW1 129.1 mm to (97.4, 159.6), turned to 0 degrees
- moved R3 127.8 mm to (92.0, 158.9), turned to 90 degrees
- moved J2 122.2 mm to (91.2, 153.1), turned to 90 degrees
- moved C7 116.4 mm to (103.0, 158.9), turned to -90 degrees
- moved D3 114.0 mm to (104.6, 167.0), turned to 0 degrees
- moved C12 112.9 mm to (105.4, 153.4), turned to 90 degrees
- moved C10 111.6 mm to (113.5, 164.5), turned to -90 degrees
- moved C14 111.1 mm to (93.8, 172.1)
- moved U1 110.3 mm to (95.2, 169.2)
- moved R4 108.3 mm to (108.4, 167.0), turned to 180 degrees
- moved C13 106.2 mm to (97.8, 163.9)
- moved C11 106.1 mm to (103.0, 162.4), turned to 90 degrees
- moved U3 105.6 mm to (109.5, 159.0), turned to 0 degrees
- moved C8 105.4 mm to (108.0, 153.0)
- moved R7 104.5 mm to (107.4, 165.0), turned to 180 degrees
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Connections:
- C10 pad 1: GND -> +3V3
- C10 pad 2: +3V0 -> GND
- C11 pad 2: +3V0 -> +3V3
- C12 pad 1: +3V0 -> +3V3
- C8 pad 2: +3V0 -> +3V3
- C9 pad 2: +3V0 -> +3V3
- J1 pad 1: GND -> SCL
- J1 pad 2: Vdd -> SDA
- J1 pad 3: SCL -> Vdd
- J1 pad 4: SDA -> GND
- J2 pad 5: SWDCLK -> SWCLK
- R3 pad 1: +3V0 -> +3V3
- R4 pad 1: Net-(U3-PB0) -> Net-(U3-PB1)
- R5 pad 1: +3V0 -> +3V3
- R6 pad 1: +3V0 -> +3V3
- R7 pad 1: Net-(U3-PB1) -> Net-(U3-PB0)
- U3 pad 1: +3V0 -> +3V3
- U3 pad 2: unconnected-(U3-PC13-Pad2) -> SWCLK
- U3 pad 24: +3V0 -> +3V3
- U3 pad 3: unconnected-(U3-PC14-Pad3) -> SWDIO
- U3 pad 34: SWDIO -> unconnected-(U3-PA13-Pad34)
- U3 pad 36: +3V0 -> +3V3
- U3 pad 37: SWDCLK -> unconnected-(U3-PA14-Pad37)
- U3 pad 48: +3V0 -> +3V3
- U3 pad 9: +3V0 -> +3V3
Routing:
- net NRST: track 54.5 -> 19.6 mm, vias 2 -> 0
- net +3V0: track 57.1 -> 23.0 mm, vias 5 -> 0
- net +3V3: track 0.00 -> 27.6 mm, vias 0 -> 6
- net Vdd: track 31.0 -> 48.9 mm, vias 0 -> 2
- net INT: track 4.21 -> 19.3 mm, vias 2 -> 0
- net SCL: track 24.8 -> 12.1 mm
- net DRDY: track 20.2 -> 7.64 mm, vias 2 -> 0
- net SWDCLK: track 10.4 -> 0.00 mm
- net GND: track 73.5 -> 63.7 mm, vias 14 -> 12
- net SDA: track 17.6 -> 10.2 mm, vias 0 -> 2
- net SWCLK: track 0.00 -> 6.46 mm
- net SWDIO: track 14.3 -> 9.52 mm
- net Net-(U3-PB1): track 2.87 -> 4.01 mm
- net Net-(U3-PB0): track 3.32 -> 2.22 mm
- net Net-(D4-A): track 2.62 -> 1.75 mm
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- added copper zone on In1.Cu, net +3V3
- added copper zone on In2.Cu, net SCL
- added copper zone on In4.Cu, net SDA
Other:
- board size 31.5 x 37.5 mm -> 34.4 x 29.6 mm
- copper layers 2 -> 6
- board text removed: "GND"
- board text removed: "RESET"
- board text removed: "SCL"
- board text removed: "SDA"
- board text removed: "SWDCLK"
- board text removed: "SWDIO"
- board text removed: "VCC"
- board text removed: "VDD"

Commit message: Finished routing
Parts:
- added C15: 10uF, Capacitor_SMD:C_0603_1608Metric_Pad1.08x0.95mm_HandSolder, F.Cu at (92.0, 174.8)
- C13: value 1uF1 -> 1uF
- C14: value 10uF1 -> 10uF
- C8: value 100nF1 -> 100nF
- moved C5 50.0 mm to (74.7, 178.6), turned to -90 degrees
- moved U5 45.2 mm to (77.2, 176.6), turned to 0 degrees
- moved C6 42.5 mm to (78.6, 178.8)
- moved R2 40.4 mm to (79.6, 174.8), turned to 90 degrees
- moved D2 38.9 mm to (77.0, 174.3)
- moved C9 36.9 mm to (81.6, 171.3), turned to -90 degrees
- moved C1 35.4 mm to (80.3, 184.8), turned to 180 degrees
- moved C10 31.0 mm to (82.5, 163.7), turned to 90 degrees
- moved C13 26.5 mm to (78.5, 182.2)
- moved U2 25.5 mm to (91.5, 180.1)
- moved R1 25.3 mm to (94.9, 179.9)
- moved R7 24.7 mm to (85.1, 175.6)
- moved D4 24.3 mm to (82.1, 175.8), turned to 90 degrees
- moved C4 24.3 mm to (89.3, 182.4), turned to -90 degrees
- moved J1 23.9 mm to (98.0, 172.6)
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Connections:
- C5 pad 1: Vdd -> +3V3
- J1 pad 3: Vdd -> +3V3
- J2 pad 2: Vdd -> +3V3
- U3 pad 2: SWCLK -> unconnected-(U3-PC13-Pad2)
- U3 pad 3: SWDIO -> unconnected-(U3-PC14-Pad3)
- U3 pad 34: unconnected-(U3-PA13-Pad34) -> SWCLK
- U3 pad 37: unconnected-(U3-PA14-Pad37) -> SWDIO
- U5 pad 1: Vdd -> +3V3
- U5 pad 3: Vdd -> +3V3
Routing:
- net Vdd: track 48.9 -> 0.00 mm, vias 2 -> 0
- net SDA: track 10.2 -> 34.7 mm, vias 2 -> 3
- net +3V0: track 23.0 -> 46.9 mm
- net SCL: track 12.1 -> 34.3 mm, vias 2 -> 3
- net +3V3: track 27.6 -> 41.0 mm, vias 6 -> 5
- net NRST: track 19.6 -> 28.4 mm
- net INT: track 19.3 -> 12.7 mm
- net SWDIO: track 9.52 -> 5.77 mm
- net SWCLK: track 6.46 -> 10.2 mm
- net Net-(U2-C1): track 1.81 -> 4.06 mm
- net Net-(U3-PB1): track 4.01 -> 1.99 mm
- net Net-(U3-PB0): track 2.22 -> 3.51 mm
- net DRDY: track 7.64 -> 6.60 mm
- net Net-(D4-A): track 1.75 -> 2.32 mm
- net GND: track 63.7 -> 63.3 mm, vias 12 -> 18
- added copper zone on F.Cu, net +3V3
- removed copper zone on F.Cu, net +3V0
- removed copper zone on In1.Cu, net +3V3
- removed copper zone on In2.Cu, net SCL
- removed copper zone on In4.Cu, net SDA
Other:
- board size 34.4 x 29.6 mm -> 28.1 x 31 mm
- copper layers 6 -> 2
