File: CTS-SAT-2-Magnetometer-Module/CTS-SAT-2-Magnetometer-Module.kicad_pcb (KiCad board)
At the start: 6 copper layers, 39.3 x 27.5 mm, 32 parts, among them J1 Conn_01x04_Pin, J2 SWD, SW1 SW_Push, U1 MMC5983MA, U2 LIS2MDL, U3 STM32F072C8Tx, U5 MIC5365-3.0YC5

Commit message: FInished routing
Other:
- board size 39.3 x 27.5 mm -> 39.3 x 26.5 mm
- board text added: "+3V3"
- board text added: "GND"
- board text added: "NRST"
- board text added: "REV 2.0"
- board text added: "SCL"
- board text added: "SDA"
- board text added: "SWCLK"
- board text added: "SWDI0"
Changed lines of the file:
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@@
 	(gr_rect
 		(start 101.077512 107.5)
-		(end 140.397753 135)
+		(end 140.397753 134)
 		(stroke
 			(width 0.05)
@@
 		(layer "Edge.Cuts")
 	)
+	(gr_text "GND"
+		(at 136.5 110.5 0)
+		(layer "B.SilkS")
+		(effects
+			(font
+				(size 1 1)
+				(thickness 0.1)
+			)
+			(justify left bottom mirror)
+		)
+	)
+	(gr_text "SDA"
+		(at 136.5 115.5 0)
+		(layer "B.SilkS")
+		(effects
+			(font
+				(size 1 1)
+				(thickness 0.1)
+			)
+			(justify left bottom mirror)
+		)
+	)
+	(gr_text "SCL"
+		(at 136.5 118 0)
+		(layer "B.SilkS")
+		(effects
+			(font
+				(size 1 1)
+				(thickness 0.1)
+			)
+			(justify left bottom mirror)
+		)
+	)
+	(gr_text "+3V3"
+		(at 137.5 113 0)
+		(layer "B.SilkS")
+		(effects
+			(font
+				(size 1 1)
+				(thickness 0.1)
+			)
+			(justify left bottom mirror)
+		)
+	)
+	(gr_text "GND"
+		(at 105.5 114 90)
+		(layer "B.SilkS")
+		(effects
+			(font
+				(size 1 1)
+				(thickness 0.1)
+			)
+			(justify left bottom mirror)
+		)
+	)
+	(gr_text "+3V3"
+		(at 108 114 90)
+		(layer "B.SilkS")
+		(effects
+			(font
+				(size 1 1)
+				(thickness 0.1)
+			)
+			(justify left bottom mirror)
+		)
+	)
+	(gr_text "NRST"
+		(at 110.5 114.5 90)
+		(layer "B.SilkS")
+		(effects
+			(font
+				(size 1 1)
+				(thickness 0.1)
+			)
+			(justify left bottom mirror)
+		)
+	)
+	(gr_text "SWDI0"
+		(at 113 114.5 90)
+		(layer "B.SilkS")
+		(effects
+			(font
+				(size 1 1)
+				(thickness 0.1)
+			)
+			(justify left bottom mirror)
+		)
+	)
+	(gr_text "SWCLK"
+		(at 115.5 114.5 90)
+		(layer "B.SilkS")
+		(effects
+			(font
+				(size 1 1)
+				(thickness 0.1)
+			)
+			(justify left bottom mirror)
+		)
+	)
+	(gr_text "REV 2.0"
+		(at 139.5 133 0)
+		(layer "B.SilkS")
+		(effects
+			(font
+				(size 1 1)
+				(thickness 0.2)
+				(bold yes)
+			)
+			(justify left bottom mirror)
+		)
+	)
 	(segment
 		(start 117.5 113.5)
@@
 	)
 	(segment
+		(start 127.4375 129.39)
+		(end 127.4375 128.4375)
+		(width 0.2)
+		(layer "F.Cu")
+		(net "DRDY")
+	)
+	(segment
+		(start 125 127.5)
+		(end 125 125.5)
+		(width 0.2)
+		(layer "F.Cu")
+		(net "DRDY")
+	)
+	(segment
 		(start 123.25 122.93241)
 		(end 123.25 122.1625)
@@
 	)
 	(segment
-		(start 127.4375 129.39)
-		(end 127.4375 128.4375)
-		(width 0.2)
-		(layer "F.Cu")
-		(net "DRDY")
-	)
-	(segment
 		(start 125.5 128)
 		(end 125 127.5)
@@
 	)
 	(segment
-		(start 123.825433 123.507843)
+		(start 123.15 123.03241)
 		(end 123.25 122.93241)
+		(width 0.2)
+		(layer "F.Cu")
+		(net "DRDY")
+	)
+	(segment
+		(start 123.15 123.65)
+		(end 123.15 123.03241)
+		(width 0.2)
+		(layer "F.Cu")
+		(net "DRDY")
+	)
+	(segment
+		(start 125 125.5)
+		(end 123.15 123.65)
+		(width 0.2)
+		(layer "F.Cu")
+		(net "DRDY")
+	)
+	(segment
+		(start 127.4375 128.4375)
+		(end 127 128)
 		(width 0.2)
 		(layer "F.Cu")
@@
 	)
 	(segment
-		(start 127.4375 128.4375)
-		(end 127 128)
-		(width 0.2)
-		(layer "F.Cu")
-		(net "DRDY")
-	)
-	(segment
-		(start 123.992157 123.507843)
-		(end 123.825433 123.507843)
-		(width 0.2)
-		(layer "F.Cu")
-		(net "DRDY")
-	)
-	(segment
-		(start 125 124.515686)
-		(end 123.992157 123.507843)
-		(width 0.2)
-		(layer "F.Cu")
-		(net "DRDY")
-	)
-	(segment
-		(start 125 127.5)
-		(end 125 124.515686)
-		(width 0.2)
-		(layer "F.Cu")
-		(net "DRDY")
-	)
-	(segment
 		(start 111.75 130.499999)
 		(end 111.75 131.25)
@@
 		(layer "F.Cu")
 		(net "Net-(D4-A)")
-	)
-	(segment
-		(start 135.3375 123.35)
-		(end 135.85 123.35)
-		(width 0.2)
-		(layer "F.Cu")
-		(net "3V3")
-	)
-	(segment
-		(start 135.3375 124.65)
-		(end 136.85 124.65)
-		(width 0.2)
-		(layer "F.Cu")
-		(net "3V3")
-	)
-	(segment
-		(start 135.85 123.35)
-		(end 137 124.5)
-		(width 0.2)
-		(layer "F.Cu")
-		(net "3V3")
-	)
-	(segment
-		(start 136.85 124.65)
-		(end 137 124.5)
-		(width 0.2)
-		(layer "F.Cu")
-		(net "3V3")
 	)
 	(segment
@@
 		(net "SWCLK")
 	)
+	(segment
+		(start 135.3375 123.35)
+		(end 135.85 123.35)
+		(width 0.2)
+		(layer "F.Cu")
+		(net "3V3")
+	)
+	(segment
+		(start 135.3375 124.65)
+		(end 136.85 124.65)
+		(width 0.2)
+		(layer "F.Cu")
+		(net "3V3")
+	)
+	(segment
+		(start 135.85 123.35)
+		(end 137 124.5)
+		(width 0.2)
+		(layer "F.Cu")
+		(net "3V3")
+	)
+	(segment
+		(start 136.85 124.65)
+		(end 137 124.5)
+		(width 0.2)
+		(layer "F.Cu")
+		(net "3V3")
+	)
 	(zone

Commit message: Fixed a label
Connections:
- C5 pad 1: 3V3 -> +3V3
- U5 pad 1: 3V3 -> +3V3
- U5 pad 3: 3V3 -> +3V3
Routing:
- net +3V3: track 87.8 -> 91.6 mm
- net 3V3: track 3.86 -> 0.00 mm
Changed lines of the file:
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@@
 			(layers "F.Cu" "F.Mask" "F.Paste")
 			(roundrect_rratio 0.25)
-			(net "3V3")
+			(net "+3V3")
 			(pinfunction "VIN_1")
 			(pintype "power_in")
@@
 			(layers "F.Cu" "F.Mask" "F.Paste")
 			(roundrect_rratio 0.25)
-			(net "3V3")
+			(net "+3V3")
 			(pinfunction "EN_3")
 			(pintype "input")
@@
 			(layers "F.Cu" "F.Mask" "F.Paste")
 			(roundrect_rratio 0.25)
-			(net "3V3")
+			(net "+3V3")
 			(pintype "passive")
 		)
@@
 	)
 	(segment
+		(start 135.3375 123.35)
+		(end 135.85 123.35)
+		(width 0.2)
+		(layer "F.Cu")
+		(net "+3V3")
+	)
+	(segment
 		(start 128 117.175)
 		(end 129.5 115.675)
@@
 	)
 	(segment
+		(start 135.3375 124.65)
+		(end 136.85 124.65)
+		(width 0.2)
+		(layer "F.Cu")
+		(net "+3V3")
+	)
+	(segment
 		(start 131.014314 112.5)
 		(end 131.217157 112.702843)
@@
 	)
 	(segment
+		(start 135.85 123.35)
+		(end 137 124.5)
+		(width 0.2)
+		(layer "F.Cu")
+		(net "+3V3")
+	)
+	(segment
 		(start 119.25 112.025)
 		(end 119.275 112)
@@
 	)
 	(segment
+		(start 136.85 124.65)
+		(end 137 124.5)
+		(width 0.2)
+		(layer "F.Cu")
+		(net "+3V3")
+	)
+	(segment
 		(start 116 122.5)
 		(end 116.5 122.5)
@@
 		(net "SWCLK")
 	)
-	(segment
-		(start 135.3375 123.35)
-		(end 135.85 123.35)
-		(width 0.2)
-		(layer "F.Cu")
-		(net "3V3")
-	)
-	(segment
-		(start 135.3375 124.65)
-		(end 136.85 124.65)
-		(width 0.2)
-		(layer "F.Cu")
-		(net "3V3")
-	)
-	(segment
-		(start 135.85 123.35)
-		(end 137 124.5)
-		(width 0.2)
-		(layer "F.Cu")
-		(net "3V3")
-	)
-	(segment
-		(start 136.85 124.65)
-		(end 137 124.5)
-		(width 0.2)
-		(layer "F.Cu")
-		(net "3V3")
-	)
 	(zone
